File: Kursa_darbs/shema.sch (KiCad schematic (older format))
At the start: 26 parts

Commit message: Pievienoti footprinti un uzlabota eeschema shēma
Parts:
- removed RV?: 10 kOhm, symbol Device:R_POT
- added J1: USB_B_Micro, symbol kursa_darbs:USB_B_Micro
- BZ1: renamed from BZ?; value TMB12A05 -> SDC1610M5; footprint (none) -> Kursa_darbs:SDC1610M5-01
- D1, D3: renamed from D?; value LED -> Red LED; footprint (none) -> Kursa_darbs:LEDC2012X90N
- D2, D5: renamed from D?; value LED -> Green LED; footprint (none) -> Kursa_darbs:LEDC2012X90N
- D4: renamed from D?; value LED -> Yellow LED; footprint (none) -> Kursa_darbs:LEDC2012X90N
- R1, R10, R11, R12, R13, R2, R3, R4, R5, R6, R7, R8, R9: renamed from R?; footprint (none) -> Kursa_darbs:RESC3216X60N
- SW1: renamed from SW?; footprint (none) -> Kursa_darbs:LL3301BF065QJ
- U1: renamed from U?; value ATmega328P -> ATmega328PB-AU; footprint Package_QFP:TQFP-32_7x7mm_P0.8mm -> Kursa_darbs:TQFP-32_7x7mm_P0.8mm; symbol MCU_Microchip_ATmega:ATmega328P-AU -> kursa_darbs:ATmega328P-AU
- U2: renamed from U?; value CD4543B -> CD4543BPWR; footprint (none) -> Kursa_darbs:CD4543B_PW_16; symbol 4xxx:4543 -> kursa_darbs:4xxx_4543
- U3: renamed from U?; value 5161AS -> SC56-11EWA; footprint Display_7Segment:SBC18-11SURKCGKWA -> Kursa_darbs:SC56-11EWA; symbol Display_Character:SBC18-11EGWA -> kursa_darbs:SBC18-11EGWA
- U4: renamed from U?; value 1602A -> REC001602AWPP5N00000; footprint Display:RC1602A -> Kursa_darbs:REC001602AWPP5N00000; symbol Display_Character:RC1602A -> kursa_darbs:shema-cache_Display_Character_RC1602A
- U5: renamed from U?; footprint (none) -> Kursa_darbs:XCVR_HC-SR04; symbol Sensor:HC-SR04 -> kursa_darbs:shema-cache_shema-rescue_HC-SR04-Sensor
Connections:
- net VCC is gone; now on net +5V: U2.1 (~LE)
- net +5V: now also J1.1 (VBUS); no longer U4.15 (A/VEE)
- net GND: now also J1.5 (GND), J1.6 (Shield); no longer U4.16 (K)
- net PB0: now reaches R8.2, U1.12 (PB0)
- net PB1: now reaches R9.2, U1.13 (PB1)
- net PB2: now reaches U1.14 (PB2), U4.5 (R/W)
- net PB3: now reaches U1.15 (PB3), U4.4 (RS)
- net PB4: now reaches U1.16 (PB4), U4.6 (E)
- net PC0: now reaches U1.23 (PC0), U4.11 (DB4)
- net PC1: now reaches U1.24 (PC1), U4.12 (DB5)
- net PC2: now reaches U1.25 (PC2), U4.13 (DB6)
- net PC3: now reaches U1.26 (PC3), U4.14 (DB7)
- net PC4: now reaches U1.27 (PC4), U5.2 (TRIG)
- net PC5: now reaches U1.28 (PC5), U5.3 (ECHO)
- net PD0: now reaches R10.2, U1.30 (PD0)
- net PD1: now reaches R11.2, U1.31 (PD1)
- net PD2: now reaches R12.2, U1.32 (PD2)
- no-connect marks 0 -> 16
Other:
- moved on the sheet: BZ1
